Commit message: Update leptrino_force_torque configuration and RViz settings; adjust force/torque ranges and visualization parameters

File: levion_arm_ros2_control/description/ros2_control/leptrino_force_torque.ros2_control.xacro (robot description, xacro)
@@ -15,10 +15,10 @@
     <state_interface name="torque.z"/>
     <param name="frame_id">tool_link</param>
-    <param name="fx_range">100</param>
-    <param name="fy_range">100</param>
-    <param name="fz_range">100</param>
-    <param name="tx_range">15</param>
-    <param name="ty_range">15</param>
-    <param name="tz_range">15</param>
+    <param name="fx_range">50</param>
+    <param name="fy_range">50</param>
+    <param name="fz_range">50</param>
+    <param name="tx_range">0.5</param>
+    <param name="ty_range">0.5</param>
+    <param name="tz_range">0.5</param>
   </sensor>
 </ros2_control>

File: levion_arm_ros2_control/description/urdf/levion_arm.urdf.xacro (robot description, xacro)
@@ -3,4 +3,5 @@
   <!-- Include ros2 control tags -->
   <xacro:include filename="$(find levion_arm_ros2_control)/ros2_control/levion_arm.ros2_control.xacro"/>
+  <xacro:include filename="$(find levion_arm_ros2_control)/ros2_control/leptrino_force_torque.ros2_control.xacro"/>
   <!-- include materials -->
   <xacro:include filename="$(find levion_arm_ros2_control)/config/material.macros.xacro"/>
@@ -67,4 +68,6 @@
     </inertial>
   </link>
+  <link name="tool_link">
+  </link>
   <joint name="world_to_link0" type="fixed">
     <origin xyz="0.08 0 0" rpy="0 0 0"/>
@@ -92,3 +95,8 @@
       velocity="${default_joint_velocity_limit}"/>
   </joint>
+  <joint name="tool_joint" type="fixed">
+    <origin xyz=".255 0 0" rpy="${PI/2} 0 ${PI/2}"/>
+    <parent link="link2"/>
+    <child link="tool_link" />
+  </joint>
 </robot>
