Commit message: Remove mirrored parameter from ak80_8_ros2_control macro calls in levion_arm.ros2_control.xacro

File: levion_arm_ros2_control/description/ros2_control/ak80_8.macros.xacro (robot description, xacro)
@@ -1,21 +1,10 @@
 <?xml version="1.0"?>
 <robot xmlns:xacro="http://ros.org/wiki/xacro">
-  <xacro:macro name="ak80_8_ros2_control" params="joint_name can_id mirrored:=false pos_min:=0.349 pos_max:=2.615 vel_limit:=10 effort_limit:=10 enc_off:=0">
-    <!-- Compute mirrored limits -->
-    <xacro:if value="${mirrored}">
-      <xacro:property name="effective_pos_min" value="${-pos_max}" />
-      <xacro:property name="effective_pos_max" value="${-pos_min}" />
-      <xacro:property name="effective_enc_off" value="${-enc_off}" />
-    </xacro:if>
-    <xacro:unless value="${mirrored}">
-      <xacro:property name="effective_pos_min" value="${pos_min}" />
-      <xacro:property name="effective_pos_max" value="${pos_max}" />
-      <xacro:property name="effective_enc_off" value="${enc_off}" />
-    </xacro:unless>
+  <xacro:macro name="ak80_8_ros2_control" params="joint_name can_id pos_min:=0.349 pos_max:=2.615 vel_limit:=10 effort_limit:=10 enc_off:=0">
     <joint name="${joint_name}">
       <!-- ros2 control basic setting -->
       <command_interface name="position">
-        <param name="min">${effective_pos_min}</param>
-        <param name="max">${effective_pos_max}</param>
+        <param name="min">${pos_min}</param>
+        <param name="max">${pos_max}</param>
       </command_interface>
       <command_interface name="velocity">
@@ -37,7 +26,7 @@
       <param name="kt">0.199</param>
       <!-- levion arm settings -->
-      <param name="pos_limit_min">${effective_pos_min}</param>
-      <param name="pos_limit_max">${effective_pos_max}</param>
-      <param name="enc_off">${effective_enc_off}</param>
+      <param name="pos_limit_min">${pos_min}</param>
+      <param name="pos_limit_max">${pos_max}</param>
+      <param name="enc_off">${enc_off}</param>
     </joint>
   </xacro:macro>

File: levion_arm_ros2_control/description/ros2_control/levion_arm.ros2_control.xacro (robot description, xacro)
@@ -15,5 +15,4 @@
       joint_name="${prefix}left_shoulder_joint"
       can_id="104"
-      mirrored="true"
       pos_min="${left_shoulder_lower}"
       pos_max="${left_shoulder_upper}"
@@ -24,5 +23,4 @@
       joint_name="${prefix}left_elbow_joint"
       can_id="105"
-      mirrored="true"
       pos_min="${left_elbow_lower}"
       pos_max="${left_elbow_upper}"
@@ -36,5 +34,4 @@
       joint_name="${prefix}right_shoulder_joint"
       can_id="204"
-      mirrored="false"
       pos_min="${right_shoulder_lower}"
       pos_max="${right_shoulder_upper}"
@@ -45,5 +42,4 @@
       joint_name="${prefix}right_elbow_joint"
       can_id="205"
-      mirrored="false"
       pos_min="${right_elbow_lower}"
       pos_max="${right_elbow_upper}"
