Commit message: Refactor levion_arm.xacro files to enable prefix argument for joint names and restructure left/right arm definitions for clarity and flexibility.

File: levion_arm_ros2_control/description/ros2_control/levion_arm.ros2_control.xacro (robot description, xacro)
@@ -1,30 +1,56 @@
 <?xml version="1.0"?>
 <robot xmlns:xacro="http://www.ros.org/wiki/xacro">
+<xacro:macro name="levion_system" params="name prefix left_arm:=true right_arm:=false">
 <!-- include macros -->
 <xacro:include filename="$(find levion_arm_ros2_control)/ros2_control/ak80_8.macros.xacro"/>
 <xacro:include filename="$(find levion_arm_ros2_control)/config/ak80_8.property.xacro"/>
-<ros2_control name="levion_arm" type="system">
+<ros2_control name="${name}" type="system">
   <hardware>
     <plugin>cubemars_hardware/CubeMarsSystemHardware</plugin>
     <param name="can_interface">can0</param>
   </hardware>
-  <xacro:ak80_8_ros2_control
-    joint_name="joint1"
-    can_id="104"
-    mirrored="true"
-    pos_min="${shoulder_joint_pos_limit_min}"
-    pos_max="${shoulder_joint_pos_limit_max}"
-    vel_limit="${default_joint_velocity_limit}"
-    effort_limit="${default_joint_effort_limit}"
-    enc_off="${shoulder_joint_encoder_offset}"/>
-  <xacro:ak80_8_ros2_control
-    joint_name="joint2"
-    can_id="105"
-    mirrored="true"
-    pos_min="${elbow_joint_pos_limit_min}"
-    pos_max="${elbow_joint_pos_limit_max}"
-    vel_limit="${default_joint_velocity_limit}"
-    effort_limit="${default_joint_effort_limit}"
-    enc_off="${elbow_joint_encoder_offset}"/>
+  <!-- Left arm -->
+  <xacro:if value="${left_arm}">
+    <xacro:ak80_8_ros2_control
+      joint_name="${prefix}left_shoulder_joint"
+      can_id="104"
+      mirrored="true"
+      pos_min="${shoulder_joint_pos_limit_min}"
+      pos_max="${shoulder_joint_pos_limit_max}"
+      vel_limit="${default_joint_velocity_limit}"
+      effort_limit="${default_joint_effort_limit}"
+      enc_off="${shoulder_joint_encoder_offset}"/>
+    <xacro:ak80_8_ros2_control
+      joint_name="${prefix}left_elbow_joint"
+      can_id="105"
+      mirrored="true"
+      pos_min="${elbow_joint_pos_limit_min}"
+      pos_max="${elbow_joint_pos_limit_max}"
+      vel_limit="${default_joint_velocity_limit}"
+      effort_limit="${default_joint_effort_limit}"
+      enc_off="${elbow_joint_encoder_offset}"/>
+  </xacro:if>
+  <!-- Right arm -->
+  <xacro:if value="${right_arm}">
+    <xacro:ak80_8_ros2_control
+      joint_name="${prefix}right_shoulder_joint"
+      can_id="204"
+      mirrored="false"
+      pos_min="${shoulder_joint_pos_limit_min}"
+      pos_max="${shoulder_joint_pos_limit_max}"
+      vel_limit="${default_joint_velocity_limit}"
+      effort_limit="${default_joint_effort_limit}"
+      enc_off="${shoulder_joint_encoder_offset}"/>
+    <xacro:ak80_8_ros2_control
+      joint_name="${prefix}right_elbow_joint"
+      can_id="205"
+      mirrored="false"
+      pos_min="${elbow_joint_pos_limit_min}"
+      pos_max="${elbow_joint_pos_limit_max}"
+      vel_limit="${default_joint_velocity_limit}"
+      effort_limit="${default_joint_effort_limit}"
+      enc_off="${elbow_joint_encoder_offset}"/>
+  </xacro:if>
 </ros2_control>
+</xacro:macro>
 </robot>

File: levion_arm_ros2_control/description/urdf/levion_arm.urdf.xacro (robot description, xacro)
@@ -1,9 +1,16 @@
 <?xml version="1.0"?>
 <robot name="levion_arm" xmlns:xacro="http://www.ros.org/wiki/xacro">
+  <!-- Enable setting arguments from the launch file -->
+  <xacro:arg name="prefix" default="" />
   <!-- Include ros2 control tags -->
   <xacro:include filename="$(find levion_arm_ros2_control)/ros2_control/levion_arm.ros2_control.xacro"/>
+  <!-- Include macros -->
+  <xacro:include filename="$(find levion_arm_ros2_control)/ros2_control/ak80_8.macros.xacro"/>
+  <xacro:include filename="$(find levion_arm_ros2_control)/config/ak80_8.property.xacro"/>
   <xacro:include filename="$(find levion_arm_ros2_control)/ros2_control/leptrino_force_torque.ros2_control.xacro"/>
   <!-- include materials -->
   <xacro:include filename="$(find levion_arm_ros2_control)/config/material.macros.xacro"/>
+  <!-- ros2 control -->
+  <xacro:levion_system name="levion_arm" prefix="" left_arm="true" right_arm="false"/>
   <!-- Main URDF -->
   <link name="world"/>

Commit message: Refactor launch and URDF files to support joint name prefixes and force torque sensor configuration; replace deprecated property file with updated version.

File: levion_arm_ros2_control/description/ros2_control/levion_arm.ros2_control.xacro (robot description, xacro)
@@ -4,5 +4,5 @@
 <!-- include macros -->
 <xacro:include filename="$(find levion_arm_ros2_control)/ros2_control/ak80_8.macros.xacro"/>
-<xacro:include filename="$(find levion_arm_ros2_control)/config/ak80_8.property.xacro"/>
+<xacro:include filename="$(find levion_arm_ros2_control)/config/levion.property.xacro"/>
 <ros2_control name="${name}" type="system">
   <hardware>
@@ -16,18 +16,18 @@
       can_id="104"
       mirrored="true"
-      pos_min="${shoulder_joint_pos_limit_min}"
-      pos_max="${shoulder_joint_pos_limit_max}"
-      vel_limit="${default_joint_velocity_limit}"
-      effort_limit="${default_joint_effort_limit}"
-      enc_off="${shoulder_joint_encoder_offset}"/>
+      pos_min="${left_shoulder_lower}"
+      pos_max="${left_shoulder_upper}"
+      vel_limit="${left_shoulder_velocity_limit}"
+      effort_limit="${left_shoulder_effort_limit}"
+      enc_off="${left_shoulder_enc_offset}"/>
     <xacro:ak80_8_ros2_control
       joint_name="${prefix}left_elbow_joint"
       can_id="105"
       mirrored="true"
-      pos_min="${elbow_joint_pos_limit_min}"
-      pos_max="${elbow_joint_pos_limit_max}"
-      vel_limit="${default_joint_velocity_limit}"
-      effort_limit="${default_joint_effort_limit}"
-      enc_off="${elbow_joint_encoder_offset}"/>
+      pos_min="${left_elbow_lower}"
+      pos_max="${left_elbow_upper}"
+      vel_limit="${left_elbow_velocity_limit}"
+      effort_limit="${left_elbow_effort_limit}"
+      enc_off="${left_elbow_enc_offset}"/>
   </xacro:if>
   <!-- Right arm -->
@@ -37,18 +37,18 @@
       can_id="204"
       mirrored="false"
-      pos_min="${shoulder_joint_pos_limit_min}"
-      pos_max="${shoulder_joint_pos_limit_max}"
-      vel_limit="${default_joint_velocity_limit}"
-      effort_limit="${default_joint_effort_limit}"
-      enc_off="${shoulder_joint_encoder_offset}"/>
+      pos_min="${right_shoulder_lower}"
+      pos_max="${right_shoulder_upper}"
+      vel_limit="${right_shoulder_velocity_limit}"
+      effort_limit="${right_shoulder_effort_limit}"
+      enc_off="${right_shoulder_enc_offset}"/>
     <xacro:ak80_8_ros2_control
       joint_name="${prefix}right_elbow_joint"
       can_id="205"
       mirrored="false"
-      pos_min="${elbow_joint_pos_limit_min}"
-      pos_max="${elbow_joint_pos_limit_max}"
-      vel_limit="${default_joint_velocity_limit}"
-      effort_limit="${default_joint_effort_limit}"
-      enc_off="${elbow_joint_encoder_offset}"/>
+      pos_min="${right_elbow_lower}"
+      pos_max="${right_elbow_upper}"
+      vel_limit="${right_elbow_velocity_limit}"
+      effort_limit="${right_elbow_effort_limit}"
+      enc_off="${right_elbow_enc_offset}"/>
   </xacro:if>
 </ros2_control>

File: levion_arm_ros2_control/description/urdf/levion_arm.macros.xacro (robot description, xacro)
@@ -2,7 +2,26 @@
 <robot xmlns:xacro="http://www.ros.org/wiki/xacro">
   <xacro:macro name="levion_arm"
-      params="parent prefix *origin left_right:=left
-      shoulder_lower shoulder_upper shoulder_vel shoulder_effort
-      elbow_lower elbow_upper elbow_vel elbow_effort">
+      params="parent prefix *origin left_right:=left">
+  <xacro:include filename="$(find levion_arm_ros2_control)/config/levion.property.xacro"/>
+  <xacro:if value="${left_right == 'left'}">
+    <xacro:property name="shoulder_lower" default="${left_shoulder_lower}" />
+    <xacro:property name="shoulder_upper" default="${left_shoulder_upper}" />
+    <xacro:property name="shoulder_vel" default="${left_shoulder_velocity_limit}" />
+    <xacro:property name="shoulder_effort" default="${left_shoulder_effort_limit}" />
+    <xacro:property name="elbow_lower" default="${left_elbow_lower}" />
+    <xacro:property name="elbow_upper" default="${left_elbow_upper}" />
+    <xacro:property name="elbow_vel" default="${left_elbow_velocity_limit}" />
+    <xacro:property name="elbow_effort" default="${left_elbow_effort_limit}" />
+  </xacro:if>
+  <xacro:if value="${left_right == 'right'}">
+    <xacro:property name="shoulder_lower" default="${right_shoulder_lower}" />
+    <xacro:property name="shoulder_upper" default="${right_shoulder_upper}" />
+    <xacro:property name="shoulder_vel" default="${right_shoulder_velocity_limit}" />
+    <xacro:property name="shoulder_effort" default="${right_shoulder_effort_limit}" />
+    <xacro:property name="elbow_lower" default="${right_elbow_lower}" />
+    <xacro:property name="elbow_upper" default="${right_elbow_upper}" />
+    <xacro:property name="elbow_vel" default="${right_elbow_velocity_limit}" />
+    <xacro:property name="elbow_effort" default="${right_elbow_effort_limit}" />
+  </xacro:if>
   <joint name="${prefix}${left_right}_base_joint" type="fixed">
     <xacro:insert_block name="origin" />

File: levion_arm_ros2_control/description/urdf/levion_arm.urdf.xacro (robot description, xacro)
@@ -3,29 +3,21 @@
   <!-- Enable setting arguments from the launch file -->
   <xacro:arg name="prefix" default="" />
-  <!-- Include ros2 control tags -->
+  <xacro:arg name="force_torque_sensor" default="true" />
+  <!-- Include materials -->
+  <xacro:include filename="$(find levion_arm_ros2_control)/config/material.macros.xacro"/>
+  <!-- Include main macros -->
+  <xacro:include filename="$(find levion_arm_ros2_control)/urdf/levion_arm.macros.xacro"/>
+  <!-- Include ros2 control macros -->
   <xacro:include filename="$(find levion_arm_ros2_control)/ros2_control/levion_arm.ros2_control.xacro"/>
-  <!-- Include macros -->
-  <xacro:include filename="$(find levion_arm_ros2_control)/config/ak80_8.property.xacro"/>
-  <xacro:include filename="$(find levion_arm_ros2_control)/urdf/levion_arm.macros.xacro"/>
-  <xacro:include filename="$(find levion_arm_ros2_control)/ros2_control/leptrino_force_torque.ros2_control.xacro"/>
-  <!-- include materials -->
-  <xacro:include filename="$(find levion_arm_ros2_control)/config/material.macros.xacro"/>
+  <xacro:if value="$(arg force_torque_sensor)">
+    <!-- Include force torque sensor macros -->
+    <!-- <xacro:include filename="$(find levion_arm_ros2_control)/ros2_control/leptrino_force_torque.ros2_control.xacro"/> -->
+  </xacro:if>
+  <!-- Main URDF -->
+  <link name="world"/>
+  <xacro:levion_arm parent="world" prefix="$(arg prefix)" left_right="left">
+    <origin xyz="0 0 0" rpy="0 0 0" />
+  </xacro:levion_arm>
   <!-- ros2 control -->
   <xacro:levion_system name="levion_arm" prefix="$(arg prefix)" left_arm="true" right_arm="true"/>
-  <!-- Main URDF -->
-  <link name="world"/>
-  <xacro:levion_arm
-    parent="world"
-    prefix="$(arg prefix)"
-    left_right="left"
-    shoulder_lower="-${default_joint_position_limit}"
-    shoulder_upper="${default_joint_position_limit}"
-    shoulder_vel="${default_joint_velocity_limit}"
-    shoulder_effort="${default_joint_effort_limit}"
-    elbow_lower="-2.615"
-    elbow_upper="-0.349"
-    elbow_vel="${default_joint_velocity_limit}"
-    elbow_effort="${default_joint_effort_limit}">
-    <origin xyz="0 0 0" rpy="0 0 0" />
-  </xacro:levion_arm>
 </robot>

Commit message: Refactor levion_system macro to conditionally include hardware plugin based on hw_plugin parameter

File: levion_arm_ros2_control/description/ros2_control/levion_arm.ros2_control.xacro (robot description, xacro)
@@ -1,13 +1,20 @@
 <?xml version="1.0"?>
 <robot xmlns:xacro="http://www.ros.org/wiki/xacro">
-<xacro:macro name="levion_system" params="name prefix left_arm:=true right_arm:=false">
+<xacro:macro name="levion_system" params="name prefix left_arm:=true right_arm:=false hw_plugin:='real'"> <!-- real/mujoco-->
 <!-- include macros -->
 <xacro:include filename="$(find levion_arm_ros2_control)/ros2_control/ak80_8.macros.xacro"/>
 <xacro:include filename="$(find levion_arm_ros2_control)/config/levion.property.xacro"/>
 <ros2_control name="${name}" type="system">
-  <hardware>
-    <plugin>cubemars_hardware/CubeMarsSystemHardware</plugin>
-    <param name="can_interface">can0</param>
-  </hardware>
+  <xacro:if value="${hw_plugin == 'real'}">
+    <hardware>
+      <plugin>cubemars_hardware/CubeMarsSystemHardware</plugin>
+      <param name="can_interface">can0</param>
+    </hardware>
+  </xacro:if>
+  <xacro:if value="${hw_plugin == 'mujoco'}">
+    <hardware>
+      <plugin>mujoco_ros2_control/MujocoSystem</plugin>
+    </hardware>
+  </xacro:if>
   <!-- Left arm -->
   <xacro:if value="${left_arm}">
