Commit message: Update joint position limits in URDF and property file for dynamic configuration

File: levion_arm_ros2_control/description/config/ak80_8.property.xacro (robot description, xacro)
@@ -9,6 +9,6 @@
   <!-- Each components -->
   <!-- Joints -->
-  <xacro:property name="shoulder_joint_pos_limit_min" value="0.349"/>
-  <xacro:property name="shoulder_joint_pos_limit_max" value="2.615"/>
+  <xacro:property name="shoulder_joint_pos_limit_min" value="-${PI}"/>
+  <xacro:property name="shoulder_joint_pos_limit_max" value="${PI}"/>
   <xacro:property name="elbow_joint_pos_limit_min" value="0.349"/>
   <xacro:property name="elbow_joint_pos_limit_max" value="2.615"/>

File: levion_arm_ros2_control/description/urdf/levion_arm.urdf.xacro (robot description, xacro)
@@ -77,5 +77,8 @@
     <child link="link1"/>
     <axis xyz="0 0 1"/>
-    <limit lower="-3.14159265359" upper="3.14159265359" effort="10" velocity="10"/>
+    <limit lower="${shoulder_joint_pos_limit_min}"
+      upper="${shoulder_joint_pos_limit_max}"
+      effort="${default_joint_effort_limit}"
+      velocity="${default_joint_velocity_limit}"/>
   </joint>
   <joint name="joint2" type="revolute">
@@ -84,5 +87,8 @@
     <child link="link2"/>
     <axis xyz="0 0 1"/>
-    <limit lower="-3.14159265359" upper="3.14159265359" effort="10" velocity="10"/>
+    <limit lower="${elbow_joint_pos_limit_min}"
+      upper="${elbow_joint_pos_limit_max}"
+      effort="${default_joint_effort_limit}"
+      velocity="${default_joint_velocity_limit}"/>
   </joint>
 </robot>

Commit message: Refactor joint position limits to use default_joint_position_limit for shoulder joints

File: levion_arm_ros2_control/description/config/ak80_8.property.xacro (robot description, xacro)
@@ -4,11 +4,11 @@
   <xacro:property name="PI" value="3.1415926535"/>
   <!-- Default -->
-  <xacro:property name="default_joint_position_limit" value="${PI}"/>
+  <xacro:property name="default_joint_position_limit" value="${PI/2}"/>
   <xacro:property name="default_joint_velocity_limit" value="10"/>
   <xacro:property name="default_joint_effort_limit" value="10"/>
   <!-- Each components -->
   <!-- Joints -->
-  <xacro:property name="shoulder_joint_pos_limit_min" value="-${PI}"/>
-  <xacro:property name="shoulder_joint_pos_limit_max" value="${PI}"/>
+  <xacro:property name="shoulder_joint_pos_limit_min" value="-${default_joint_position_limit}"/>
+  <xacro:property name="shoulder_joint_pos_limit_max" value="${default_joint_position_limit}"/>
   <xacro:property name="elbow_joint_pos_limit_min" value="0.349"/>
   <xacro:property name="elbow_joint_pos_limit_max" value="2.615"/>
