Commit message: Add encoder offset parameters for shoulder and elbow joints in Xacro files

File: levion_arm_ros2_control/description/config/ak80_8.macros.xacro (robot description, xacro)
@@ -1,5 +1,5 @@
 <?xml version="1.0"?>
 <robot xmlns:xacro="http://ros.org/wiki/xacro">
-  <xacro:macro name="ak80_8_ros2_control" params="joint_name can_id pos_min:=0.349 pos_max:=2.615 vel_limit:=10 effort_limit:=10">
+  <xacro:macro name="ak80_8_ros2_control" params="joint_name can_id pos_min:=0.349 pos_max:=2.615 vel_limit:=10 effort_limit:=10 enc_off:=0">
     <joint name="${joint_name}">
       <!-- ros2 control basic setting -->
@@ -28,4 +28,5 @@
       <param name="pos_limit_min">${pos_min}</param>
       <param name="pos_limit_max">${pos_max}</param>
+      <param name="enc_off">${enc_off}</param>
     </joint>
   </xacro:macro>

File: levion_arm_ros2_control/description/config/ak80_8.property.xacro (robot description, xacro)
@@ -11,6 +11,8 @@
   <xacro:property name="shoulder_joint_pos_limit_min" value="-${default_joint_position_limit}"/>
   <xacro:property name="shoulder_joint_pos_limit_max" value="${default_joint_position_limit}"/>
+  <xacro:property name="shoulder_joint_encoder_offset" value="0"/>
   <xacro:property name="elbow_joint_pos_limit_min" value="0.349"/>
   <xacro:property name="elbow_joint_pos_limit_max" value="2.615"/>
+  <xacro:property name="elbow_joint_encoder_offset" value="0.349"/>
   <!-- Links -->
 </robot>

File: levion_arm_ros2_control/description/ros2_control/levion_arm.ros2_control.xacro (robot description, xacro)
@@ -15,5 +15,6 @@
     pos_max="${shoulder_joint_pos_limit_max}"
     vel_limit="${default_joint_velocity_limit}"
-    effort_limit="${default_joint_effort_limit}"/>
+    effort_limit="${default_joint_effort_limit}"
+    enc_off="${shoulder_joint_encoder_offset}"/>
   <xacro:ak80_8_ros2_control
     joint_name="joint2"
@@ -22,5 +23,6 @@
     pos_max="${elbow_joint_pos_limit_max}"
     vel_limit="${default_joint_velocity_limit}"
-    effort_limit="${default_joint_effort_limit}"/>
+    effort_limit="${default_joint_effort_limit}"
+    enc_off="${elbow_joint_encoder_offset}"/>
 </ros2_control>
 </robot>

Commit message: Update ak80_8 macros and properties to support mirrored joint configurations

File: levion_arm_ros2_control/description/config/ak80_8.macros.xacro (robot description, xacro)
@@ -1,10 +1,20 @@
 <?xml version="1.0"?>
 <robot xmlns:xacro="http://ros.org/wiki/xacro">
-  <xacro:macro name="ak80_8_ros2_control" params="joint_name can_id pos_min:=0.349 pos_max:=2.615 vel_limit:=10 effort_limit:=10 enc_off:=0">
+  <xacro:macro name="ak80_8_ros2_control" params="joint_name can_id mirrored:=false pos_min:=0.349 pos_max:=2.615 vel_limit:=10 effort_limit:=10 enc_off:=0">
+    <!-- Compute mirrored limits -->
+    <xacro:if value="${mirrored}">
+      <xacro:property name="effective_pos_min" value="$((-1.0 * pos_max))" />
+      <xacro:property name="effective_pos_max" value="$((-1.0 * pos_min))" />
+      <xacro:property name="effective_enc_off" value="$((-1.0 * enc_off))" />
+    </xacro:if>
+    <xacro:unless value="${mirrored}">
+      <xacro:property name="effective_pos_min" value="${pos_min}" />
+      <xacro:property name="effective_pos_max" value="${pos_max}" />
+    </xacro:unless>
     <joint name="${joint_name}">
       <!-- ros2 control basic setting -->
       <command_interface name="position">
-        <param name="min">${pos_min}</param>
-        <param name="max">${pos_max}</param>
+        <param name="min">${effective_pos_min}</param>
+        <param name="max">${effective_pos_max}</param>
       </command_interface>
       <command_interface name="velocity">
@@ -26,7 +36,7 @@
       <param name="kt">0.199</param>
       <!-- levion arm settings -->
-      <param name="pos_limit_min">${pos_min}</param>
-      <param name="pos_limit_max">${pos_max}</param>
-      <param name="enc_off">${enc_off}</param>
+      <param name="pos_limit_min">${effective_pos_min}</param>
+      <param name="pos_limit_max">${effective_pos_max}</param>
+      <param name="enc_off">${effective_enc_off}</param>
     </joint>
   </xacro:macro>

File: levion_arm_ros2_control/description/config/ak80_8.property.xacro (robot description, xacro)
@@ -14,5 +14,5 @@
   <xacro:property name="elbow_joint_pos_limit_min" value="0.349"/>
   <xacro:property name="elbow_joint_pos_limit_max" value="2.615"/>
-  <xacro:property name="elbow_joint_encoder_offset" value="0.349"/>
+  <xacro:property name="elbow_joint_encoder_offset" value="-0.349"/>
   <!-- Links -->
 </robot>

Commit message: Add effective encoder offset property for non-mirrored joint configurations

File: levion_arm_ros2_control/description/config/ak80_8.macros.xacro (robot description, xacro)
@@ -11,4 +11,5 @@
       <xacro:property name="effective_pos_min" value="${pos_min}" />
       <xacro:property name="effective_pos_max" value="${pos_max}" />
+      <xacro:property name="effective_enc_off" value="${enc_off}" />
     </xacro:unless>
     <joint name="${joint_name}">

Commit message: Refactor mirrored limit calculations for clarity and consistency

File: levion_arm_ros2_control/description/config/ak80_8.macros.xacro (robot description, xacro)
@@ -4,7 +4,7 @@
     <!-- Compute mirrored limits -->
     <xacro:if value="${mirrored}">
-      <xacro:property name="effective_pos_min" value="$((-1.0 * pos_max))" />
-      <xacro:property name="effective_pos_max" value="$((-1.0 * pos_min))" />
-      <xacro:property name="effective_enc_off" value="$((-1.0 * enc_off))" />
+      <xacro:property name="effective_pos_min" value="${-pos_max}" />
+      <xacro:property name="effective_pos_max" value="${-pos_min}" />
+      <xacro:property name="effective_enc_off" value="${-enc_off}" />
     </xacro:if>
     <xacro:unless value="${mirrored}">
