Commit message: Enhance JointVelocityGui to dynamically subscribe to joint states and publish velocities based on slider inputs

File: levion_arm_ros2_control/description/config/levion.property.xacro (robot description, xacro)
@@ -3,4 +3,10 @@
   <!-- Math -->
   <xacro:property name="PI" value="3.1415926535"/>
+  <xacro:property name="PI_2" value="${PI/2}"/>
+  <xacro:property name="PI_4" value="${PI/4}"/>
+  <xacro:property name="SQRT2" value="1.4142135623"/>
+  <xacro:property name="SQRT2_2" value="${SQRT2/2}"/>
+  <xacro:property name="SQRT3" value="1.7320508076"/>
+  <xacro:property name="SQRT3_2" value="${SQRT3/2}"/>
   <!-- Default -->
   <xacro:property name="default_joint_position_limit" value="${PI/2}"/>

Commit message: Update joint position limits to incorporate safety offset for elbow joints

File: levion_arm_ros2_control/description/config/levion.property.xacro (robot description, xacro)
@@ -9,6 +9,7 @@
   <xacro:property name="SQRT3" value="1.7320508076"/>
   <xacro:property name="SQRT3_2" value="${SQRT3/2}"/>
+  <xacro:property name="SAFETY_OFFSET" value="0.01"/>
   <!-- Default -->
-  <xacro:property name="default_joint_position_limit" value="${PI/2}"/>
+  <xacro:property name="default_joint_position_limit" value="${PI/2-SAFETY_OFFSET}"/>
   <xacro:property name="default_joint_velocity_limit" value="10"/>
   <xacro:property name="default_joint_effort_limit" value="10"/>
@@ -16,6 +17,6 @@
   <xacro:property name="shoulder_upper" value="${default_joint_position_limit}"/>
   <xacro:property name="shoulder_enc_offset" value="0"/>
-  <xacro:property name="elbow_lower" value="-2.615"/>
-  <xacro:property name="elbow_upper" value="-0.349"/>
+  <xacro:property name="elbow_lower" value="-2.615+SAFETY_OFFSET"/>
+  <xacro:property name="elbow_upper" value="-0.349-SAFETY_OFFSET"/>
   <xacro:property name="elbow_enc_offset" value="0.349"/>
   <!-- Left joints -->

Commit message: Fix elbow joint limits to correctly apply safety offset in property file

File: levion_arm_ros2_control/description/config/levion.property.xacro (robot description, xacro)
@@ -17,6 +17,6 @@
   <xacro:property name="shoulder_upper" value="${default_joint_position_limit}"/>
   <xacro:property name="shoulder_enc_offset" value="0"/>
-  <xacro:property name="elbow_lower" value="-2.615+SAFETY_OFFSET"/>
-  <xacro:property name="elbow_upper" value="-0.349-SAFETY_OFFSET"/>
+  <xacro:property name="elbow_lower" value="${-2.615+SAFETY_OFFSET}"/>
+  <xacro:property name="elbow_upper" value="${-0.349-SAFETY_OFFSET}"/>
   <xacro:property name="elbow_enc_offset" value="0.349"/>
   <!-- Left joints -->
