Commit message: Update STL mesh files for Link0, Link1, and Link2; modify RViz fixed frame to 'world' and adjust URDF for world link and joint definitions

File: levion_arm_ros2_control/description/urdf/levion_arm.urdf.xacro (robot description, xacro)
@@ -4,7 +4,8 @@
   <xacro:include filename="$(find levion_arm_ros2_control)/ros2_control/ak80_8.ros2_control.xacro"/>
   <!-- Main URDF -->
+  <link name="world"/>
   <link name="link0">
-    <origin xyz="0 0 0" rpy="${PI} 0 0"/>
     <visual>
+      <origin xyz="0 0 0" rpy="0 0 0"/>
       <geometry>
         <mesh filename="file://$(find levion_arm_ros2_control)/mesh/Link0.STL" scale="1 1 1"/>
@@ -42,6 +43,11 @@
     </inertial>
   </link>
+  <joint name="world_to_link0" type="fixed">
+    <origin xyz="0 -0.000 0" rpy="0 0 0"/>
+    <parent link="world"/>
+    <child link="link0"/>
+  </joint>
   <joint name="ak80_8_joint" type="revolute">
-    <origin xyz="0 0 0.03" rpy="0 0 0"/>
+    <origin xyz="0 0 0" rpy="0 0 0"/>
     <parent link="link0"/>
     <child link="link1"/>

Commit message: Add mesh files for Link1 and Link2; update URDF for visual and collision geometry

File: levion_arm_ros2_control/description/urdf/levion_arm.urdf.xacro (robot description, xacro)
@@ -34,5 +34,24 @@
       <origin xyz="0 0 0" rpy="0 0 0"/>
       <geometry>
-        <cylinder radius=".04" length="0.01"/>
+        <mesh filename="file://$(find levion_arm_ros2_control)/mesh/Link1.STL" scale="1 1 1"/>
+      </geometry>
+    </collision>
+    <inertial>
+      <origin xyz="0 0 0" rpy="0 0 0"/>
+      <mass value="0.1"/>
+      <inertia ixx="0.0001" ixy="0.0" ixz="0.0" iyy="0.0001" iyz="0.0" izz="0.0001"/>
+    </inertial>
+  </link>
+  <link name="link2">
+    <visual>
+      <origin xyz="0 0 0" rpy="0 0 0"/>
+      <geometry>
+        <mesh filename="file://$(find levion_arm_ros2_control)/mesh/Link2.STL" scale="1 1 1"/>
+      </geometry>
+    </visual>
+    <collision>
+      <origin xyz="0 0 0" rpy="0 0 0"/>
+      <geometry>
+        <mesh filename="file://$(find levion_arm_ros2_control)/mesh/Link2.STL" scale="1 1 1"/>
       </geometry>
     </collision>
@@ -44,10 +63,10 @@
   </link>
   <joint name="world_to_link0" type="fixed">
-    <origin xyz="0 -0.000 0" rpy="0 0 0"/>
+    <origin xyz="0.08 0 0" rpy="0 0 0"/>
     <parent link="world"/>
     <child link="link0"/>
   </joint>
-  <joint name="ak80_8_joint" type="revolute">
-    <origin xyz="0 0 0" rpy="0 0 0"/>
+  <joint name="joint1" type="revolute">
+    <origin xyz="0 0 0.0439" rpy="0 0 0"/>
     <parent link="link0"/>
     <child link="link1"/>
@@ -55,3 +74,10 @@
     <limit lower="-3.14159265359" upper="3.14159265359" effort="10" velocity="10"/>
   </joint>
+  <joint name="joint2" type="revolute">
+    <origin xyz="0.32 0 0.04685" rpy="0 0 0"/>
+    <parent link="link1"/>
+    <child link="link2"/>
+    <axis xyz="0 0 1"/>
+    <limit lower="-3.14159265359" upper="3.14159265359" effort="10" velocity="10"/>
+  </joint>
 </robot>

Commit message: Add material macros and update URDF to include levion_black for visual elements of links

File: levion_arm_ros2_control/description/urdf/levion_arm.urdf.xacro (robot description, xacro)
@@ -2,5 +2,7 @@
 <robot name="ak80_8" xmlns:xacro="http://www.ros.org/wiki/xacro">
   <!-- Include ros2 control tags -->
-  <xacro:include filename="$(find levion_arm_ros2_control)/ros2_control/ak80_8.ros2_control.xacro"/>
+  <xacro:include filename="$(find levion_arm_ros2_control)/ros2_control/levion_arm.ros2_control.xacro"/>
+  <!-- include materials -->
+  <xacro:include filename="$(find levion_arm_ros2_control)/config/material.macros.xacro"/>
   <!-- Main URDF -->
   <link name="world"/>
@@ -9,6 +11,7 @@
       <origin xyz="0 0 0" rpy="0 0 0"/>
       <geometry>
-        <mesh filename="file://$(find levion_arm_ros2_control)/mesh/Link0.STL" scale="1 1 1"/>
+        <mesh filename="file://$(find levion_arm_ros2_control)/mesh/Link0.STL" scale="1 1 1" color="0. 0. 0."/>
       </geometry>
+      <xacro:levion_black/>
     </visual>
     <collision>
@@ -30,4 +33,5 @@
         <mesh filename="file://$(find levion_arm_ros2_control)/mesh/Link1.STL" scale="1 1 1"/>
       </geometry>
+      <xacro:levion_black/>
     </visual>
     <collision>
@@ -49,4 +53,5 @@
         <mesh filename="file://$(find levion_arm_ros2_control)/mesh/Link2.STL" scale="1 1 1"/>
       </geometry>
+      <xacro:levion_black/>
     </visual>
     <collision>

Commit message: Refactor levion_arm.urdf.xacro to include new levion_arm macros and update joint parameters for improved flexibility and configuration.

File: levion_arm_ros2_control/description/urdf/levion_arm.urdf.xacro (robot description, xacro)
@@ -6,104 +6,26 @@
   <xacro:include filename="$(find levion_arm_ros2_control)/ros2_control/levion_arm.ros2_control.xacro"/>
   <!-- Include macros -->
-  <xacro:include filename="$(find levion_arm_ros2_control)/ros2_control/ak80_8.macros.xacro"/>
   <xacro:include filename="$(find levion_arm_ros2_control)/config/ak80_8.property.xacro"/>
+  <xacro:include filename="$(find levion_arm_ros2_control)/urdf/levion_arm.macros.xacro"/>
   <xacro:include filename="$(find levion_arm_ros2_control)/ros2_control/leptrino_force_torque.ros2_control.xacro"/>
   <!-- include materials -->
   <xacro:include filename="$(find levion_arm_ros2_control)/config/material.macros.xacro"/>
   <!-- ros2 control -->
-  <xacro:levion_system name="levion_arm" prefix="" left_arm="true" right_arm="false"/>
+  <xacro:levion_system name="levion_arm" prefix="$(arg prefix)" left_arm="true" right_arm="true"/>
   <!-- Main URDF -->
   <link name="world"/>
-  <link name="link0">
-    <visual>
-      <origin xyz="0 0 0" rpy="0 0 0"/>
-      <geometry>
-        <mesh filename="file://$(find levion_arm_ros2_control)/mesh/Link0.STL" scale="1 1 1" color="0. 0. 0."/>
-      </geometry>
-      <xacro:levion_black/>
-    </visual>
-    <collision>
-      <origin xyz="0 0 0" rpy="0 0 0"/>
-      <geometry>
-        <mesh filename="file://$(find levion_arm_ros2_control)/mesh/Link0.STL" scale="1 1 1"/>
-      </geometry>
-    </collision>
-    <inertial>
-      <origin xyz="0 0 0" rpy="0 0 0"/>
-      <mass value="0.1"/>
-      <inertia ixx="0.0001" ixy="0.0" ixz="0.0" iyy="0.0001" iyz="0.0" izz="0.0001"/>
-    </inertial>
-  </link>
-  <link name="link1">
-    <visual>
-      <origin xyz="0 0 0" rpy="0 0 0"/>
-      <geometry>
-        <mesh filename="file://$(find levion_arm_ros2_control)/mesh/Link1.STL" scale="1 1 1"/>
-      </geometry>
-      <xacro:levion_black/>
-    </visual>
-    <collision>
-      <origin xyz="0 0 0" rpy="0 0 0"/>
-      <geometry>
-        <mesh filename="file://$(find levion_arm_ros2_control)/mesh/Link1.STL" scale="1 1 1"/>
-      </geometry>
-    </collision>
-    <inertial>
-      <origin xyz="0 0 0" rpy="0 0 0"/>
-      <mass value="0.1"/>
-      <inertia ixx="0.0001" ixy="0.0" ixz="0.0" iyy="0.0001" iyz="0.0" izz="0.0001"/>
-    </inertial>
-  </link>
-  <link name="link2">
-    <visual>
-      <origin xyz="0 0 0" rpy="0 0 0"/>
-      <geometry>
-        <mesh filename="file://$(find levion_arm_ros2_control)/mesh/Link2.STL" scale="1 1 1"/>
-      </geometry>
-      <xacro:levion_black/>
-    </visual>
-    <collision>
-      <origin xyz="0 0 0" rpy="0 0 0"/>
-      <geometry>
-        <mesh filename="file://$(find levion_arm_ros2_control)/mesh/Link2.STL" scale="1 1 1"/>
-      </geometry>
-    </collision>
-    <inertial>
-      <origin xyz="0 0 0" rpy="0 0 0"/>
-      <mass value="0.1"/>
-      <inertia ixx="0.0001" ixy="0.0" ixz="0.0" iyy="0.0001" iyz="0.0" izz="0.0001"/>
-    </inertial>
-  </link>
-  <link name="tool_link">
-  </link>
-  <joint name="world_to_link0" type="fixed">
-    <origin xyz="0.08 0 0" rpy="0 0 0"/>
-    <parent link="world"/>
-    <child link="link0"/>
-  </joint>
-  <joint name="joint1" type="revolute">
-    <origin xyz="0 0 0.0439" rpy="0 0 0"/>
-    <parent link="link0"/>
-    <child link="link1"/>
-    <axis xyz="0 0 1"/>
-    <limit lower="${shoulder_joint_pos_limit_min}"
-      upper="${shoulder_joint_pos_limit_max}"
-      effort="${default_joint_effort_limit}"
-      velocity="${default_joint_velocity_limit}"/>
-  </joint>
-  <joint name="joint2" type="revolute">
-    <origin xyz="0.32 0 0.04685" rpy="0 0 0"/>
-    <parent link="link1"/>
-    <child link="link2"/>
-    <axis xyz="0 0 1"/>
-    <limit lower="${elbow_joint_pos_limit_min}"
-      upper="${elbow_joint_pos_limit_max}"
-      effort="${default_joint_effort_limit}"
-      velocity="${default_joint_velocity_limit}"/>
-  </joint>
-  <joint name="tool_joint" type="fixed">
-    <origin xyz=".255 0 0" rpy="${PI/2} 0 ${PI/2}"/>
-    <parent link="link2"/>
-    <child link="tool_link" />
-  </joint>
+  <xacro:levion_arm
+    parent="world"
+    prefix="$(arg prefix)"
+    left_right="left"
+    shoulder_lower="-${default_joint_position_limit}"
+    shoulder_upper="${default_joint_position_limit}"
+    shoulder_vel="${default_joint_velocity_limit}"
+    shoulder_effort="${default_joint_effort_limit}"
+    elbow_lower="-2.615"
+    elbow_upper="-0.349"
+    elbow_vel="${default_joint_velocity_limit}"
+    elbow_effort="${default_joint_effort_limit}">
+    <origin xyz="0 0 0" rpy="0 0 0" />
+  </xacro:levion_arm>
 </robot>

Commit message: Remove redundant right arm definition from levion_arm.urdf.xacro for clarity and consistency.

File: levion_arm_ros2_control/description/urdf/levion_arm.urdf.xacro (robot description, xacro)
@@ -19,7 +19,4 @@
     <origin xyz="0 0 0" rpy="0 0 0" />
   </xacro:levion_arm>
-  <xacro:levion_arm parent="world" prefix="$(arg prefix)" left_right="right">
-    <origin xyz="0 0 0" rpy="0 0 0" />
-  </xacro:levion_arm>
   <!-- ros2 control -->
   <xacro:levion_system name="levion_arm" prefix="$(arg prefix)" left_arm="true" right_arm="true"/>
