Commit message: Refactor levion_arm macros and URDF to ensure consistent naming conventions for links and joints; add missing right arm definition in URDF.

File: levion_arm_ros2_control/description/urdf/levion_arm.macros.xacro (robot description, xacro)
@@ -27,7 +27,7 @@
     <xacro:insert_block name="origin" />
     <parent link="${parent}"/>
-    <child link="${prefix}${left_right}link0" />
+    <child link="${prefix}${left_right}_link0" />
   </joint>
-  <link name="${prefix}${left_right}link0">
+  <link name="${prefix}${left_right}_link0">
     <visual>
       <origin xyz="0 0 0" rpy="0 0 0"/>
@@ -49,5 +49,5 @@
     </inertial>
   </link>
-  <link name="${prefix}${left_right}link1">
+  <link name="${prefix}${left_right}_link1">
     <visual>
       <origin xyz="0 0 0" rpy="0 0 0"/>
@@ -69,5 +69,5 @@
     </inertial>
   </link>
-  <link name="${prefix}${left_right}link2">
+  <link name="${prefix}${left_right}_link2">
     <visual>
       <origin xyz="0 0 0" rpy="0 0 0"/>
@@ -89,10 +89,10 @@
     </inertial>
   </link>
-  <link name="${prefix}${left_right}tool_link">
+  <link name="${prefix}${left_right}_tool_link">
   </link>
-  <joint name="${prefix}${left_right}shoulder_joint" type="revolute">
+  <joint name="${prefix}${left_right}_shoulder_joint" type="revolute">
     <origin xyz="0 0 0.0439" rpy="0 0 0"/>
-    <parent link="${prefix}${left_right}link0"/>
-    <child link="${prefix}${left_right}link1"/>
+    <parent link="${prefix}${left_right}_link0"/>
+    <child link="${prefix}${left_right}_link1"/>
     <axis xyz="0 0 1"/>
     <limit lower="${shoulder_lower}"
@@ -101,8 +101,8 @@
       velocity="${shoulder_vel}"/>
   </joint>
-  <joint name="${prefix}${left_right}elbow_joint" type="revolute">
+  <joint name="${prefix}${left_right}_elbow_joint" type="revolute">
     <origin xyz="0.32 0 0.04685" rpy="0 0 0"/>
-    <parent link="${prefix}${left_right}link1"/>
-    <child link="${prefix}${left_right}link2"/>
+    <parent link="${prefix}${left_right}_link1"/>
+    <child link="${prefix}${left_right}_link2"/>
     <axis xyz="0 0 1"/>
     <limit lower="${elbow_lower}"
@@ -111,8 +111,8 @@
       velocity="${elbow_vel}"/>
   </joint>
-  <joint name="${prefix}${left_right}tool_joint" type="fixed">
+  <joint name="${prefix}${left_right}_tool_joint" type="fixed">
     <origin xyz=".255 0 0" rpy="${PI/2} 0 ${PI/2}"/>
-    <parent link="${prefix}${left_right}link2"/>
-    <child link="${prefix}${left_right}tool_link"/>
+    <parent link="${prefix}${left_right}_link2"/>
+    <child link="${prefix}${left_right}_tool_link"/>
   </joint>
   </xacro:macro>

File: levion_arm_ros2_control/description/urdf/levion_arm.urdf.xacro (robot description, xacro)
@@ -19,4 +19,7 @@
     <origin xyz="0 0 0" rpy="0 0 0" />
   </xacro:levion_arm>
+  <xacro:levion_arm parent="world" prefix="$(arg prefix)" left_right="right">
+    <origin xyz="0 0 0" rpy="0 0 0" />
+  </xacro:levion_arm>
   <!-- ros2 control -->
   <xacro:levion_system name="levion_arm" prefix="$(arg prefix)" left_arm="true" right_arm="true"/>

Commit message: Refactor levion_arm macros to standardize shoulder and elbow property names with 'lr_' prefix for consistency across left and right arm definitions.

File: levion_arm_ros2_control/description/urdf/levion_arm.macros.xacro (robot description, xacro)
@@ -5,22 +5,22 @@
   <xacro:include filename="$(find levion_arm_ros2_control)/config/levion.property.xacro"/>
   <xacro:if value="${left_right == 'left'}">
-    <xacro:property name="shoulder_lower" default="${left_shoulder_lower}" />
-    <xacro:property name="shoulder_upper" default="${left_shoulder_upper}" />
-    <xacro:property name="shoulder_vel" default="${left_shoulder_velocity_limit}" />
-    <xacro:property name="shoulder_effort" default="${left_shoulder_effort_limit}" />
-    <xacro:property name="elbow_lower" default="${left_elbow_lower}" />
-    <xacro:property name="elbow_upper" default="${left_elbow_upper}" />
-    <xacro:property name="elbow_vel" default="${left_elbow_velocity_limit}" />
-    <xacro:property name="elbow_effort" default="${left_elbow_effort_limit}" />
+    <xacro:property name="lr_shoulder_lower" default="${left_shoulder_lower}" />
+    <xacro:property name="lr_shoulder_upper" default="${left_shoulder_upper}" />
+    <xacro:property name="lr_shoulder_vel" default="${left_shoulder_velocity_limit}" />
+    <xacro:property name="lr_shoulder_effort" default="${left_shoulder_effort_limit}" />
+    <xacro:property name="lr_elbow_lower" default="${left_elbow_lower}" />
+    <xacro:property name="lr_elbow_upper" default="${left_elbow_upper}" />
+    <xacro:property name="lr_elbow_vel" default="${left_elbow_velocity_limit}" />
+    <xacro:property name="lr_elbow_effort" default="${left_elbow_effort_limit}" />
   </xacro:if>
   <xacro:if value="${left_right == 'right'}">
-    <xacro:property name="shoulder_lower" default="${right_shoulder_lower}" />
-    <xacro:property name="shoulder_upper" default="${right_shoulder_upper}" />
-    <xacro:property name="shoulder_vel" default="${right_shoulder_velocity_limit}" />
-    <xacro:property name="shoulder_effort" default="${right_shoulder_effort_limit}" />
-    <xacro:property name="elbow_lower" default="${right_elbow_lower}" />
-    <xacro:property name="elbow_upper" default="${right_elbow_upper}" />
-    <xacro:property name="elbow_vel" default="${right_elbow_velocity_limit}" />
-    <xacro:property name="elbow_effort" default="${right_elbow_effort_limit}" />
+    <xacro:property name="lr_shoulder_lower" default="${right_shoulder_lower}" />
+    <xacro:property name="lr_shoulder_upper" default="${right_shoulder_upper}" />
+    <xacro:property name="lr_shoulder_vel" default="${right_shoulder_velocity_limit}" />
+    <xacro:property name="lr_shoulder_effort" default="${right_shoulder_effort_limit}" />
+    <xacro:property name="lr_elbow_lower" default="${right_elbow_lower}" />
+    <xacro:property name="lr_elbow_upper" default="${right_elbow_upper}" />
+    <xacro:property name="lr_elbow_vel" default="${right_elbow_velocity_limit}" />
+    <xacro:property name="lr_elbow_effort" default="${right_elbow_effort_limit}" />
   </xacro:if>
   <joint name="${prefix}${left_right}_base_joint" type="fixed">
@@ -96,8 +96,8 @@
     <child link="${prefix}${left_right}_link1"/>
     <axis xyz="0 0 1"/>
-    <limit lower="${shoulder_lower}"
-      upper="${shoulder_upper}"
-      effort="${shoulder_effort}"
-      velocity="${shoulder_vel}"/>
+    <limit lower="${lr_shoulder_lower}"
+      upper="${lr_shoulder_upper}"
+      effort="${lr_shoulder_effort}"
+      velocity="${lr_shoulder_vel}"/>
   </joint>
   <joint name="${prefix}${left_right}_elbow_joint" type="revolute">
@@ -106,8 +106,8 @@
     <child link="${prefix}${left_right}_link2"/>
     <axis xyz="0 0 1"/>
-    <limit lower="${elbow_lower}"
-      upper="${elbow_upper}"
-      effort="${elbow_effort}"
-      velocity="${elbow_vel}"/>
+    <limit lower="${lr_elbow_lower}"
+      upper="${lr_elbow_upper}"
+      effort="${lr_elbow_effort}"
+      velocity="${lr_elbow_vel}"/>
   </joint>
   <joint name="${prefix}${left_right}_tool_joint" type="fixed">

Commit message: Update controller name and adjust velocity scaling in JointVelocityGui

File: levion_arm_ros2_control/description/urdf/levion_arm.macros.xacro (robot description, xacro)
@@ -33,5 +33,5 @@
       <origin xyz="0 0 0" rpy="0 0 0"/>
       <geometry>
-        <mesh filename="file://$(find levion_arm_ros2_control)/mesh/Link0.STL" scale="1 1 1" color="0. 0. 0."/>
+        <mesh filename="package://levion_arm_ros2_control/mesh/Link0.STL" scale="1 1 1"/>
       </geometry>
       <xacro:levion_black/>
@@ -40,5 +40,5 @@
       <origin xyz="0 0 0" rpy="0 0 0"/>
       <geometry>
-        <mesh filename="file://$(find levion_arm_ros2_control)/mesh/Link0.STL" scale="1 1 1"/>
+        <mesh filename="package://levion_arm_ros2_control/mesh/Link0.STL" scale="1 1 1"/>
       </geometry>
     </collision>
@@ -53,5 +53,5 @@
       <origin xyz="0 0 0" rpy="0 0 0"/>
       <geometry>
-        <mesh filename="file://$(find levion_arm_ros2_control)/mesh/Link1.STL" scale="1 1 1"/>
+        <mesh filename="package://levion_arm_ros2_control/mesh/Link1.STL" scale="1 1 1"/>
       </geometry>
       <xacro:levion_black/>
@@ -60,5 +60,5 @@
       <origin xyz="0 0 0" rpy="0 0 0"/>
       <geometry>
-        <mesh filename="file://$(find levion_arm_ros2_control)/mesh/Link1.STL" scale="1 1 1"/>
+        <mesh filename="package://levion_arm_ros2_control/mesh/Link1.STL" scale="1 1 1"/>
       </geometry>
     </collision>
@@ -73,5 +73,5 @@
       <origin xyz="0 0 0" rpy="0 0 0"/>
       <geometry>
-        <mesh filename="file://$(find levion_arm_ros2_control)/mesh/Link2.STL" scale="1 1 1"/>
+        <mesh filename="package://levion_arm_ros2_control/mesh/Link2.STL" scale="1 1 1"/>
       </geometry>
       <xacro:levion_black/>
@@ -80,5 +80,5 @@
       <origin xyz="0 0 0" rpy="0 0 0"/>
       <geometry>
-        <mesh filename="file://$(find levion_arm_ros2_control)/mesh/Link2.STL" scale="1 1 1"/>
+        <mesh filename="package://levion_arm_ros2_control/mesh/Link2.STL" scale="1 1 1"/>
       </geometry>
     </collision>

Commit message: Update inertial properties for levion arm links to reflect accurate mass and inertia values

File: levion_arm_ros2_control/description/urdf/levion_arm.macros.xacro (robot description, xacro)
@@ -45,6 +45,6 @@
     <inertial>
       <origin xyz="0 0 0" rpy="0 0 0"/>
-      <mass value="0.1"/>
-      <inertia ixx="0.0001" ixy="0.0" ixz="0.0" iyy="0.0001" iyz="0.0" izz="0.0001"/>
+      <mass value="0.5"/>
+      <inertia ixx="0.0005" ixy="0.0" ixz="0.0" iyy="0.0005" iyz="0.0" izz="0.0005"/>
     </inertial>
   </link>
@@ -64,7 +64,7 @@
     </collision>
     <inertial>
-      <origin xyz="0 0 0" rpy="0 0 0"/>
-      <mass value="0.1"/>
-      <inertia ixx="0.0001" ixy="0.0" ixz="0.0" iyy="0.0001" iyz="0.0" izz="0.0001"/>
+      <origin xyz="0.05 0 0" rpy="0 0 0"/>
+      <mass value="0.6"/>
+      <inertia ixx="0.0006" ixy="0.0" ixz="0.0" iyy="0.0006" iyz="0.0" izz="0.0006"/>
     </inertial>
   </link>
